Commit message: adds initial multi bot sim effort

File: description/gazebo_control.xacro (robot description, xacro)
@@ -2,5 +2,8 @@
 <robot xmlns:xacro="http://www.ros.org/wiki/xacro" >
     <gazebo>
-        <plugin name="diff_drive" filename="libgazebo_ros_diff_drive.so">
+        <plugin filename="libgazebo_ros_diff_drive.so" name="diff_drive">
+            <ros>
+        <!-- <namespace>/pathfinder</namespace> -->
+            </ros>
             <!-- Wheel Information -->
             <left_joint>left_wheel_joint</left_joint>

File: description/robot_core.xacro (robot description, xacro)
@@ -1,4 +1,4 @@
 <?xml version="1.0"?>
-<robot name="pathfinder" xmlns:xacro="http://www.ros.org/wiki/xacro" >
+<robot xmlns:xacro="http://www.ros.org/wiki/xacro" >
     <!--includes-->
     <xacro:include filename="inertial_macros.xacro"/>
@@ -17,5 +17,5 @@
             <origin xyz="0.15 0 0" rpy="0 0 ${pi/2}"/>
             <geometry>
-                <mesh filename="file://$(find pathfinder)/description/meshes/pathfinder_chassis.stl" scale="0.001 0.001 0.001"/>
+                <mesh filename="file://$(find pathfinder)/description/meshes/pathfinder_chassis.stl" scale="0.001 0.001 0.001"/> <!-- scale is in meters -->
             </geometry>
             <material name="fontys_purple"/>
