Commit message: adds gazebo control pkg

File: description/robot.urdf.xacro (robot description, xacro)
@@ -2,3 +2,4 @@
 <robot name="pathfinder" xmlns:xacro="http://www.ros.org/wiki/xacro" >
     <xacro:include filename="robot_core.xacro" />
+    <xacro:include filename="gazebo_control.xacro" />
 </robot>

File: description/robot_core.xacro (robot description, xacro)
@@ -105,3 +105,8 @@
         </xacro:inertial_sphere>
     </link>
+    <gazebo reference="caster_wheel">
+        <material>Gazebo/Black</material>
+        <mu1 value="0.001"/> <!-- friction -->
+        <mu2 value="0.001"/>
+    </gazebo>
 </robot>

Commit message: fixes error parsing urdf xml string

File: description/robot.urdf.xacro (robot description, xacro)
@@ -1,4 +1,4 @@
 <?xml version="1.0"?>
-<robot xmlns:xacro="http://www.ros.org/wiki/xacro" >
+<robot name="pathfinder" xmlns:xacro="http://www.ros.org/wiki/xacro" >
     <xacro:include filename="robot_core.xacro" />
     <xacro:include filename="gazebo_control.xacro" />

File: description/robot_core.xacro (robot description, xacro)
@@ -6,4 +6,12 @@
     <!-- BASE LINK -->
     <link name="base_link">
+    </link>
+     <!-- BASE FOOTPRINT LINK -->
+    <joint name="base_footprint_joint" type="fixed">
+        <parent link="base_link"/>
+        <child link="chassis"/>
+        <origin xyz="0 0 0" rpy="0 0 0"/>
+    </joint>
+    <link name="base_footprint">
     </link>
     <!-- CHASSIS LINK -->
