Commit message: adds lidar sensor

File: description/materials.xacro (robot description, xacro)
@@ -8,5 +8,8 @@
         <color rgba="0 0 0 1"/>
     </material>
-     <material name="fontys_purple">
+    <material name="red">
+        <color rgba="1 0 0 1"/>
+    </material>
+    <material name="fontys_purple">
         <color rgba="${102/255} ${51/255} ${102/255} 1"/>
     </material>

File: description/robot.urdf.xacro (robot description, xacro)
@@ -3,3 +3,4 @@
     <xacro:include filename="robot_core.xacro" />
     <xacro:include filename="gazebo_control.xacro" />
+    <xacro:include filename="lidar.xacro" />
 </robot>

Commit message: format urdf

File: description/materials.xacro (robot description, xacro)
@@ -11,4 +11,10 @@
         <color rgba="1 0 0 1"/>
     </material>
+    <material name="green">
+        <color rgba="0 1 0 1"/>
+    </material>
+    <material name="blue">
+        <color rgba="0 0 1 1"/>
+    </material>
     <material name="fontys_purple">
         <color rgba="${102/255} ${51/255} ${102/255} 1"/>
