Commit message: adds branded pathfinder_chassis.stl

File: description/robot_core.xacro (robot description, xacro)
@@ -1,16 +1,18 @@
 <?xml version="1.0"?>
 <robot xmlns:xacro="http://www.ros.org/wiki/xacro" >
+    <!--includes-->
     <xacro:include filename="inertial_macros.xacro"/>
+    <!--materials-->
     <material name="white">
         <color rgba="1 1 1 1" />
     </material>
-    <material name="orange">
-        <color rgba="1 0.3 0.1 1"/>
+    <material name="black">
+        <color rgba="0 0 0 1"/>
+    </material>
+     <material name="fontys_purple">
+        <color rgba="${102/255} ${51/255} ${102/255} 1"/>
     </material>
     <material name="blue">
         <color rgba="0.2 0.2 1 1"/>
-    </material>
-    <material name="black">
-        <color rgba="0 0 0 1"/>
     </material>
     <!-- BASE LINK -->
@@ -27,7 +29,7 @@
             <origin xyz="0.15 0 0.075"/>
             <geometry>
-                <box size="0.3 0.3 0.15"/>
+                <mesh filename="package://description/meshes/pathfinder_chassis.stl" scale="1 1 1"/>
             </geometry>
-            <material name="white"/>
+            <material name="fontys_purple"/>
         </visual>
         <collision>
@@ -53,5 +55,5 @@
                 <cylinder radius="0.05" length="0.04"/>
             </geometry>
-            <material name="blue"/>
+            <material name="black"/>
         </visual>
         <collision>
@@ -76,5 +78,5 @@
                 <cylinder radius="0.05" length="0.04"/>
             </geometry>
-            <material name="blue"/>
+            <material name="black"/>
         </visual>
         <collision>

Commit message: fixes meshes file path

File: description/robot_core.xacro (robot description, xacro)
@@ -29,5 +29,5 @@
             <origin xyz="0.15 0 0.075"/>
             <geometry>
-                <mesh filename="package://description/meshes/pathfinder_chassis.stl" scale="1 1 1"/>
+                <mesh filename="package://meshes/pathfinder_chassis.stl" scale="1 1 1"/>
             </geometry>
             <material name="fontys_purple"/>

Commit message: fixes file path

File: description/robot_core.xacro (robot description, xacro)
@@ -29,5 +29,5 @@
             <origin xyz="0.15 0 0.075"/>
             <geometry>
-                <mesh filename="package://meshes/pathfinder_chassis.stl" scale="1 1 1"/>
+                <mesh filename="package://pathfinder/descriptions/meshes/pathfinder_chassis.stl" scale="1 1 1"/>
             </geometry>
             <material name="fontys_purple"/>

Commit message: adds robot name to description

File: description/robot_core.xacro (robot description, xacro)
@@ -1,4 +1,4 @@
 <?xml version="1.0"?>
-<robot xmlns:xacro="http://www.ros.org/wiki/xacro" >
+<robot name="pathfinder" xmlns:xacro="http://www.ros.org/wiki/xacro" >
     <!--includes-->
     <xacro:include filename="inertial_macros.xacro"/>
@@ -29,5 +29,5 @@
             <origin xyz="0.15 0 0.075"/>
             <geometry>
-                <mesh filename="package://pathfinder/descriptions/meshes/pathfinder_chassis.stl" scale="1 1 1"/>
+                <mesh filename="package://pathfinder/description/meshes/pathfinder_chassis.stl" scale="1 1 1"/>
             </geometry>
             <material name="fontys_purple"/>

Commit message: fix the stl mesh path

File: description/robot_core.xacro (robot description, xacro)
@@ -29,5 +29,5 @@
             <origin xyz="0.15 0 0.075"/>
             <geometry>
-                <mesh filename="package://pathfinder/description/meshes/pathfinder_chassis.stl" scale="1 1 1"/>
+                <mesh filename="package://description/meshes/pathfinder_chassis.stl" scale="1.0 1.0 1.0"/>
             </geometry>
             <material name="fontys_purple"/>

Commit message: change mesh import syntax to ros2

File: description/robot_core.xacro (robot description, xacro)
@@ -29,5 +29,5 @@
             <origin xyz="0.15 0 0.075"/>
             <geometry>
-                <mesh filename="package://description/meshes/pathfinder_chassis.stl" scale="1.0 1.0 1.0"/>
+                <mesh filename="file://$(find pathfinder)/description/meshes/pathfinder_chassis.stl" scale="1.0 1.0 1.0"/>
             </geometry>
             <material name="fontys_purple"/>

Commit message: adds robot name to all xacro files

File: description/robot_core.xacro (robot description, xacro)
@@ -29,5 +29,5 @@
             <origin xyz="0.15 0 0.075"/>
             <geometry>
-                <mesh filename="file://$(find pathfinder)/description/meshes/pathfinder_chassis.stl" scale="1.0 1.0 1.0"/>
+                <mesh filename="file://$(find pathfinder)/src/description/meshes/pathfinder_chassis.stl" scale="1.0 1.0 1.0"/>
             </geometry>
             <material name="fontys_purple"/>

Commit message: final fix for chassis stl path

File: description/robot_core.xacro (robot description, xacro)
@@ -29,5 +29,5 @@
             <origin xyz="0.15 0 0.075"/>
             <geometry>
-                <mesh filename="file://$(find pathfinder)/src/description/meshes/pathfinder_chassis.stl" scale="1.0 1.0 1.0"/>
+                <mesh filename="file://$(find pathfinder)/description/meshes/pathfinder_chassis.stl" scale="1.0 1.0 1.0"/>
             </geometry>
             <material name="fontys_purple"/>

Commit message: changes mesh scaling to correct size

File: description/robot_core.xacro (robot description, xacro)
@@ -29,5 +29,5 @@
             <origin xyz="0.15 0 0.075"/>
             <geometry>
-                <mesh filename="file://$(find pathfinder)/description/meshes/pathfinder_chassis.stl" scale="1.0 1.0 1.0"/>
+                <mesh filename="file://$(find pathfinder)/description/meshes/pathfinder_chassis.stl" scale="0.001 0.001 0.001"/>
             </geometry>
             <material name="fontys_purple"/>

Commit message: change pitch

File: description/robot_core.xacro (robot description, xacro)
@@ -27,5 +27,5 @@
     <link name="chassis">
         <visual>
-            <origin xyz="0.15 0 0.075"/>
+            <origin xyz="0.15 0 0" rpy="0 ${pi/4} 0"/>
             <geometry>
                 <mesh filename="file://$(find pathfinder)/description/meshes/pathfinder_chassis.stl" scale="0.001 0.001 0.001"/>

Commit message: change yaw

File: description/robot_core.xacro (robot description, xacro)
@@ -27,5 +27,5 @@
     <link name="chassis">
         <visual>
-            <origin xyz="0.15 0 0" rpy="0 ${pi/4} 0"/>
+            <origin xyz="0.15 0 0" rpy="0 0 ${pi/4}"/>
             <geometry>
                 <mesh filename="file://$(find pathfinder)/description/meshes/pathfinder_chassis.stl" scale="0.001 0.001 0.001"/>

Commit message: final origin

File: description/robot_core.xacro (robot description, xacro)
@@ -27,5 +27,5 @@
     <link name="chassis">
         <visual>
-            <origin xyz="0.15 0 0" rpy="0 0 ${pi/4}"/>
+            <origin xyz="0.15 0 0" rpy="0 0 ${pi/2}"/>
             <geometry>
                 <mesh filename="file://$(find pathfinder)/description/meshes/pathfinder_chassis.stl" scale="0.001 0.001 0.001"/>

Commit message: adds gazebo launch file

File: description/robot_core.xacro (robot description, xacro)
@@ -3,17 +3,5 @@
     <!--includes-->
     <xacro:include filename="inertial_macros.xacro"/>
-    <!--materials-->
-    <material name="white">
-        <color rgba="1 1 1 1" />
-    </material>
-    <material name="black">
-        <color rgba="0 0 0 1"/>
-    </material>
-     <material name="fontys_purple">
-        <color rgba="${102/255} ${51/255} ${102/255} 1"/>
-    </material>
-    <material name="blue">
-        <color rgba="0.2 0.2 1 1"/>
-    </material>
+    <xacro:include filename="materials.xacro"/>
     <!-- BASE LINK -->
     <link name="base_link">
@@ -66,4 +54,7 @@
         </xacro:inertial_cylinder>
     </link>
+    <gazebo reference="left_wheel">
+        <material>Gazebo/Black</material>
+    </gazebo>
     <!-- RIGHT WHEEL LINK -->
     <joint name="right_wheel_joint" type="continuous">
@@ -89,4 +80,7 @@
         </xacro:inertial_cylinder>
     </link>
+    <gazebo reference="right_wheel">
+        <material>Gazebo/Black</material>
+    </gazebo>
     <!-- CASTER WHEEL LINK -->
     <joint name="caster_wheel_joint" type="fixed">

Commit message: sets correct child link to base footprint

File: description/robot_core.xacro (robot description, xacro)
@@ -10,5 +10,5 @@
     <joint name="base_footprint_joint" type="fixed">
         <parent link="base_link"/>
-        <child link="chassis"/>
+        <child link="base_footprint"/>
         <origin xyz="0 0 0" rpy="0 0 0"/>
     </joint>

Commit message: remove footprint for now

File: description/robot_core.xacro (robot description, xacro)
@@ -7,5 +7,5 @@
     <link name="base_link">
     </link>
-     <!-- BASE FOOTPRINT LINK -->
+     <!-- BASE FOOTPRINT LINK
     <joint name="base_footprint_joint" type="fixed">
         <parent link="base_link"/>
@@ -14,5 +14,5 @@
     </joint>
     <link name="base_footprint">
-    </link>
+    </link> -->
     <!-- CHASSIS LINK -->
     <joint name="chassis_joint" type="fixed">

Commit message: removes footprint

File: description/robot_core.xacro (robot description, xacro)
@@ -8,5 +8,5 @@
     </link>
      <!-- BASE FOOTPRINT LINK -->
-    <joint name="base_footprint_joint" type="fixed">
+    <!-- <joint name="base_footprint_joint" type="fixed">
         <parent link="base_link"/>
         <child link="base_footprint"/>
@@ -14,5 +14,5 @@
     </joint>
     <link name="base_footprint">
-    </link>
+    </link> -->
     <!-- CHASSIS LINK -->
     <joint name="chassis_joint" type="fixed">
