Commit message: directory structure changes

File: description/gazebo_lidar.xacro (robot description, xacro)
@@ -4,5 +4,5 @@
         <parent link="chassis"/>
         <child link="laser_frame"/>
-        <origin xyz="0.1 0 0.175" rpy="0 0 0"/>
+        <origin xyz="0.1 0 0.12" rpy="0 0 0"/>
     </joint>
     <link name="laser_frame">

Commit message: moves lidar to original postion

File: description/gazebo_lidar.xacro (robot description, xacro)
@@ -4,5 +4,5 @@
         <parent link="chassis"/>
         <child link="laser_frame"/>
-        <origin xyz="0.1 0 0.12" rpy="0 0 0"/>
+        <origin xyz="0.1 0 0.16" rpy="0 0 0"/>
     </joint>
     <link name="laser_frame">
