Commit message: change depth cam position

File: description/depth_camera.xacro (robot description, xacro)
@@ -15,5 +15,5 @@
             <origin xyz="0.15 0 0.075"/>
             <geometry>
-                <box size="0.3 0.3 0.15"/>
+                <box size="0.03 0.03 0.02"/>
             </geometry>
         </collision>
@@ -22,5 +22,5 @@
         <parent link="camera_link"/>
         <child link="camera_link_optical"/>
-        <origin xyz="0 0 0" rpy="${-pi/2} 0 ${-pi/2}"/>
+        <origin xyz="0 0 0" rpy="${-pi/2} 0 ${-pi/3}"/>
     </joint>
     <link name="camera_link_optical"></link>

Commit message: change d435 position

File: description/depth_camera.xacro (robot description, xacro)
@@ -4,5 +4,5 @@
         <parent link="chassis"/>
         <child link="camera_link"/>
-        <origin xyz="0.32 0 0.1" rpy="0 0 0"/>
+        <origin xyz="0.32 0 0.1" rpy="0 0 ${-pi/2}"/>
     </joint>
     <link name="camera_link">
@@ -13,7 +13,7 @@
         </visual>
         <collision>
-            <origin xyz="0.15 0 0.075"/>
+            <origin xyz="0 0 0"/>
             <geometry>
-                <box size="0.03 0.03 0.02"/>
+              <mesh filename="file://$(find pathfinder)/description/meshes/intel_realsense_D435.stl" scale="0.001 0.001 0.001"/> <!-- scale is in meters -->
             </geometry>
         </collision>
@@ -22,5 +22,5 @@
         <parent link="camera_link"/>
         <child link="camera_link_optical"/>
-        <origin xyz="0 0 0" rpy="${-pi/2} 0 ${-pi/3}"/>
+        <origin xyz="0 0 0" rpy="${-pi/2} 0 ${-pi/2}"/>
     </joint>
     <link name="camera_link_optical"></link>

Commit message: minor format changes

File: description/depth_camera.xacro (robot description, xacro)
@@ -9,11 +9,14 @@
         <visual>
             <geometry>
-               <mesh filename="file://$(find pathfinder)/description/meshes/intel_realsense_D435.stl" scale="0.001 0.001 0.001"/> <!-- scale is in meters -->
+              <mesh filename="file://$(find pathfinder)/description/meshes/intel_realsense_D435.stl"
+                        scale="0.001 0.001 0.001"/> <!-- scale is in meters -->
             </geometry>
+            <material name="blue"/>
         </visual>
         <collision>
             <origin xyz="0 0 0"/>
             <geometry>
-              <mesh filename="file://$(find pathfinder)/description/meshes/intel_realsense_D435.stl" scale="0.001 0.001 0.001"/> <!-- scale is in meters -->
+              <mesh filename="file://$(find pathfinder)/description/meshes/intel_realsense_D435.stl"
+                    scale="0.001 0.001 0.001"/> <!-- scale is in meters -->
             </geometry>
         </collision>
@@ -35,5 +38,5 @@
                 <image>
                     <format>B8G8R8</format>
-                    <width>640</width>
+                    <width>848</width>
                     <height>480</height>
                 </image>

Commit message: fix camera origin

File: description/depth_camera.xacro (robot description, xacro)
@@ -25,5 +25,5 @@
         <parent link="camera_link"/>
         <child link="camera_link_optical"/>
-        <origin xyz="0 0 0" rpy="${-pi/2} 0 ${-pi/2}"/>
+        <origin xyz="0 0 0" rpy="0 0 ${-pi/2}"/>
     </joint>
     <link name="camera_link_optical"></link>

Commit message: change the camera position and collision

File: description/depth_camera.xacro (robot description, xacro)
@@ -4,8 +4,9 @@
         <parent link="chassis"/>
         <child link="camera_link"/>
-        <origin xyz="0.32 0 0.1" rpy="0 0 ${-pi/2}"/>
+        <origin xyz="0.3 0 0.1" rpy="0 0 ${-pi/2}"/>
     </joint>
     <link name="camera_link">
         <visual>
+            <origin xyz="0 0 0" rpy="0 0 0"/>
             <geometry>
               <mesh filename="file://$(find pathfinder)/description/meshes/intel_realsense_D435.stl"
@@ -15,5 +16,5 @@
         </visual>
         <collision>
-            <origin xyz="0 0 0"/>
+            <origin xyz="0.3 0 0.1" rpy="0 0 0"/>
             <geometry>
               <mesh filename="file://$(find pathfinder)/description/meshes/intel_realsense_D435.stl"

File: description/robot_core.xacro (robot description, xacro)
@@ -11,5 +11,5 @@
         <parent link="base_link"/>
         <child link="base_footprint"/>
-        <origin xyz="0 0 0" rpy="0 0 0"/>
+        <origin xyz="0 0 -0.05" rpy="0 0 0"/>
     </joint>
     <link name="base_footprint">

Commit message: sets correct camera origin

File: description/depth_camera.xacro (robot description, xacro)
@@ -4,5 +4,5 @@
         <parent link="chassis"/>
         <child link="camera_link"/>
-        <origin xyz="0.3 0 0.1" rpy="0 0 ${-pi/2}"/>
+        <origin xyz="0.31 0 0.1" rpy="0 0 ${-pi/2}"/>
     </joint>
     <link name="camera_link">
@@ -16,5 +16,5 @@
         </visual>
         <collision>
-            <origin xyz="0.3 0 0.1" rpy="0 0 0"/>
+            <origin xyz="0 0 0" rpy="0 0 0"/>
             <geometry>
               <mesh filename="file://$(find pathfinder)/description/meshes/intel_realsense_D435.stl"

Commit message: fixes camera yaw

File: description/depth_camera.xacro (robot description, xacro)
@@ -26,5 +26,5 @@
         <parent link="camera_link"/>
         <child link="camera_link_optical"/>
-        <origin xyz="0 0 0" rpy="0 0 ${-pi/2}"/>
+        <origin xyz="0 0 0" rpy="0 0 0"/>
     </joint>
     <link name="camera_link_optical"></link>

Commit message: change the camera optical joint roll

File: description/depth_camera.xacro (robot description, xacro)
@@ -26,5 +26,5 @@
         <parent link="camera_link"/>
         <child link="camera_link_optical"/>
-        <origin xyz="0 0 0" rpy="0 0 0"/>
+        <origin xyz="0 0 0" rpy="${-pi/2} 0 0"/>
     </joint>
     <link name="camera_link_optical"></link>
@@ -39,5 +39,5 @@
                 <image>
                     <format>B8G8R8</format>
-                    <width>848</width>
+                    <width>640</width>
                     <height>480</height>
                 </image>

Commit message: adds inertial properties to camera

File: description/depth_camera.xacro (robot description, xacro)
@@ -4,5 +4,5 @@
         <parent link="chassis"/>
         <child link="camera_link"/>
-        <origin xyz="0.31 0 0.1" rpy="0 0 ${-pi/2}"/>
+        <origin xyz="0.3125 0 0.1" rpy="0 0 ${-pi/2}"/>
     </joint>
     <link name="camera_link">
@@ -22,9 +22,12 @@
             </geometry>
         </collision>
+         <xacro:inertial_box mass="0.1" x="0.025" y="0.09" z="0.025">
+            <origin xyz="0 0 0.0" rpy="0 0 0"/>
+        </xacro:inertial_box>
     </link>
     <joint name="camera_optical_joint" type="fixed">
         <parent link="camera_link"/>
         <child link="camera_link_optical"/>
-        <origin xyz="0 0 0" rpy="${-pi/2} 0 0"/>
+        <origin xyz="0 0 0" rpy="${-pi/2} 0 0"/> <!-- rotate 90 degrees around x-axis. Z axis becomes depth(x-axis)-->
     </joint>
     <link name="camera_link_optical"></link>
@@ -43,12 +46,12 @@
                 </image>
                 <clip>
-                    <near>0.15</near>
-                    <far>8.0</far>
+                    <near>0.28</near>
+                    <far>6.0</far>
                 </clip>
             </camera>
             <plugin name="camera_controller" filename="libgazebo_ros_camera.so">
                 <frame_name>camera_link_optical</frame_name>
-                <min_depth>0.1</min_depth>
-                <max_depth>100.0</max_depth>
+                <min_depth>0.28</min_depth>
+                <max_depth>6.0</max_depth>
             </plugin>
         </sensor>

Commit message: fix segmentation error

File: description/depth_camera.xacro (robot description, xacro)
@@ -4,5 +4,5 @@
         <parent link="chassis"/>
         <child link="camera_link"/>
-        <origin xyz="0.3125 0 0.1" rpy="0 0 ${-pi/2}"/>
+        <origin xyz="0.31 0 0.1" rpy="0 0 ${-pi/2}"/>
     </joint>
     <link name="camera_link">

File: description/gazebo_lidar.xacro (robot description, xacro)
@@ -43,5 +43,5 @@
             <plugin name="laser_controller" filename="libgazebo_ros_ray_sensor.so">
                 <ros>
-                    <argument>~/out:=scan</argument>
+                    <argument>--ros-args --remap ~/out:=scan</argument>
                 </ros>
                 <output_type>sensor_msgs/LaserScan</output_type>

File: description/robot_core.xacro (robot description, xacro)
@@ -7,5 +7,5 @@
     <link name="base_link">
     </link>
-     <!-- BASE FOOTPRINT LINK
+     <!-- BASE FOOTPRINT LINK -->
     <joint name="base_footprint_joint" type="fixed">
         <parent link="base_link"/>
@@ -14,5 +14,5 @@
     </joint>
     <link name="base_footprint">
-    </link> -->
+    </link>
     <!-- CHASSIS LINK -->
     <joint name="chassis_joint" type="fixed">

Commit message: minor changes to improve stability

File: description/depth_camera.xacro (robot description, xacro)
@@ -29,5 +29,5 @@
         <parent link="camera_link"/>
         <child link="camera_link_optical"/>
-        <origin xyz="0 0 0" rpy="${-pi/2} 0 0"/> <!-- rotate 90 degrees around x-axis. Z axis becomes depth(x-axis)-->
+        <origin xyz="0 0 0" rpy="${-pi/2} 0 ${-pi/2}"/> <!-- rotate 90 degrees around x-axis. Z axis becomes depth(x-axis)-->
     </joint>
     <link name="camera_link_optical"></link>

File: description/robot.urdf.xacro (robot description, xacro)
@@ -4,4 +4,4 @@
     <xacro:include filename="gazebo_control.xacro" />
     <xacro:include filename="gazebo_lidar.xacro" />
-    <xacro:include filename="depth_camera.xacro" />
+    <!-- <xacro:include filename="depth_camera.xacro" /> -->
 </robot>

File: description/robot_core.xacro (robot description, xacro)
@@ -8,5 +8,5 @@
     </link>
      <!-- BASE FOOTPRINT LINK -->
-    <!-- <joint name="base_footprint_joint" type="fixed">
+    <joint name="base_footprint_joint" type="fixed">
         <parent link="base_link"/>
         <child link="base_footprint"/>
@@ -14,5 +14,5 @@
     </joint>
     <link name="base_footprint">
-    </link> -->
+    </link>
     <!-- CHASSIS LINK -->
     <joint name="chassis_joint" type="fixed">

Commit message: final fixes

File: description/depth_camera.xacro (robot description, xacro)
@@ -4,9 +4,9 @@
         <parent link="chassis"/>
         <child link="camera_link"/>
-        <origin xyz="0.31 0 0.1" rpy="0 0 ${-pi/2}"/>
+        <origin xyz="0.31 0 0.1" rpy="0 0 0"/>
     </joint>
     <link name="camera_link">
         <visual>
-            <origin xyz="0 0 0" rpy="0 0 0"/>
+            <origin xyz="0 0 0" rpy="0 0 ${-pi/2}"/>
             <geometry>
               <mesh filename="file://$(find pathfinder)/description/meshes/intel_realsense_D435.stl"
@@ -18,6 +18,5 @@
             <origin xyz="0 0 0" rpy="0 0 0"/>
             <geometry>
-              <mesh filename="file://$(find pathfinder)/description/meshes/intel_realsense_D435.stl"
-                    scale="0.001 0.001 0.001"/> <!-- scale is in meters -->
+                <box size="0.025 0.09 0.025"/>
             </geometry>
         </collision>

Commit message: big overhaul

File: description/depth_camera.xacro (robot description, xacro)
@@ -4,5 +4,5 @@
         <parent link="chassis"/>
         <child link="camera_link"/>
-        <origin xyz="0.31 0 0.1" rpy="0 0 0"/>
+        <origin xyz="0.305 0 0.1" rpy="0 0 0"/>
     </joint>
     <link name="camera_link">
@@ -28,5 +28,5 @@
         <parent link="camera_link"/>
         <child link="camera_link_optical"/>
-        <origin xyz="0 0 0" rpy="${-pi/2} 0 ${-pi/2}"/> <!-- rotate 90 degrees around x-axis. Z axis becomes depth(x-axis)-->
+        <origin xyz="0 0 0" rpy="${-pi/2} 0 ${-pi/2}"/> <!-- Z axis becomes depth(x-axis)-->
     </joint>
     <link name="camera_link_optical"></link>

File: description/gazebo_control.xacro (robot description, xacro)
@@ -2,8 +2,8 @@
 <robot xmlns:xacro="http://www.ros.org/wiki/xacro" >
     <gazebo>
-        <plugin filename="libgazebo_ros_diff_drive.so" name="diff_drive">
+        <plugin name="diff_drive" filename="libgazebo_ros_diff_drive.so">
             <ros>
-               <!--<namespace>-->
-               <!--<remapping tf>-->
+               <!--<namespace> added during multi bot launch </namespace>-->
+               <!--<remapping> added during multi bot launch </remapping>-->
             </ros>
             <!-- Wheel Information -->

File: description/gazebo_lidar.xacro (robot description, xacro)
@@ -11,5 +11,5 @@
                 <cylinder radius="0.05" length="0.04"/>
             </geometry>
-            <material name="red"/>
+            <material name="blue"/>
         </visual>
         <collision>
@@ -23,8 +23,8 @@
     </link>
     <gazebo reference="laser_frame">
-        <material>Gazebo/Red</material>
+        <material>Gazebo/Blue</material>
         <sensor name="laser" type="ray">
             <pose> 0 0 0 0 0 0 </pose>
-            <visualize>true</visualize>
+            <visualize>false</visualize>
             <update_rate>10</update_rate>
             <ray>
@@ -38,10 +38,10 @@
                 <range>
                     <min>0.3</min>
-                    <max>10</max>
+                    <max>12</max>
                 </range>
             </ray>
             <plugin name="laser_controller" filename="libgazebo_ros_ray_sensor.so">
                 <ros>
-                    <argument>~/out:=scan</argument>
+                    <remapping>~/out:=scan</remapping>
                 </ros>
                 <output_type>sensor_msgs/LaserScan</output_type>

File: description/materials.xacro (robot description, xacro)
@@ -17,4 +17,7 @@
         <color rgba="0 0 1 1"/>
     </material>
+    <material name="grey">
+        <color rgba="${128/255} ${128/255} ${128/255} 1"/>
+    </material>
     <material name="fontys_purple">
         <color rgba="${102/255} ${51/255} ${102/255} 1"/>

File: description/robot_core.xacro (robot description, xacro)
@@ -39,4 +39,7 @@
         </xacro:inertial_box>
     </link>
+    <gazebo reference="chassis">
+        <material>Gazebo/Purple</material>
+    </gazebo>
     <!-- LEFT WHEEL LINK -->
     <joint name="left_wheel_joint" type="continuous">
@@ -102,5 +105,5 @@
                 <sphere radius="0.05"/>
             </geometry>
-            <material name="black"/>
+            <material name="grey"/>
         </visual>
         <collision>
@@ -114,5 +117,5 @@
     </link>
     <gazebo reference="caster_wheel">
-        <material>Gazebo/Black</material>
+        <material>Gazebo/Grey</material>
         <mu1 value="0.001"/> <!-- friction -->
         <mu2 value="0.001"/>

Commit message: adds depth camera

File: description/depth_camera.xacro (robot description, xacro)
@@ -4,5 +4,5 @@
         <parent link="chassis"/>
         <child link="camera_link"/>
-        <origin xyz="0.305 0 0.1" rpy="0 0 0"/>
+        <origin xyz="0.31 0 0.1" rpy="0 0 0"/>
     </joint>
     <link name="camera_link">
@@ -35,8 +35,8 @@
         <sensor name="camera" type="depth">
             <pose> 0 0 0 0 0 0 </pose>
-            <visualize>true</visualize>
-            <update_rate>10</update_rate>
+            <visualize>false</visualize>
+            <update_rate>15</update_rate>
             <camera>
-                <horizontal_fov>1.089</horizontal_fov>
+                <!-- <horizontal_fov>1.089</horizontal_fov> -->
                 <image>
                     <format>B8G8R8</format>
@@ -46,5 +46,5 @@
                 <clip>
                     <near>0.28</near>
-                    <far>6.0</far>
+                    <far>10.0</far>
                 </clip>
             </camera>

File: description/gazebo_lidar.xacro (robot description, xacro)
@@ -4,5 +4,5 @@
         <parent link="chassis"/>
         <child link="laser_frame"/>
-        <origin xyz="0.1 0 0.16" rpy="0 0 0"/>
+        <origin xyz="0.1 0 0.17" rpy="0 0 0"/>
     </joint>
     <link name="laser_frame">
@@ -26,5 +26,5 @@
         <sensor name="laser" type="ray">
             <pose> 0 0 0 0 0 0 </pose>
-            <visualize>true</visualize>
+            <visualize>false</visualize>
             <update_rate>20</update_rate>
             <ray>

File: description/robot.urdf.xacro (robot description, xacro)
@@ -4,4 +4,4 @@
     <xacro:include filename="gazebo_control.xacro" />
     <xacro:include filename="gazebo_lidar.xacro" />
-    <!-- <xacro:include filename="depth_camera.xacro" /> -->
+    <xacro:include filename="depth_camera.xacro" />
 </robot>
